File: rubber_ducky.kicad_pcb (KiCad board)
At the start: 2 copper layers, 14 parts, among them U1 ATmega32U4-A, U2 USB-C-2.0, Y1 ASCO

Commit message: usbc fix
Parts:
- moved U2 2.83 mm to (138.2, 81.5)
- moved R2 1.39 mm to (143.5, 85.1)
- moved R1 1.33 mm to (143.5, 87.3)
Routing:
- net GND: track 13.6 -> 9.77 mm
- net /D+: track 5.01 -> 7.31 mm
- net /D1+: track 9.27 -> 7.06 mm
- net /D-: track 5.42 -> 7.31 mm
- net /D1-: track 8.89 -> 7.33 mm
- added copper zone on B.Cu, net GND
