File: rubber_ducky.kicad_pcb (KiCad board)
At the start: 2 copper layers, 36.7 x 18.7 mm, 15 parts, among them U1 ATmega32U4-A, U2 USB-C-2.0, Y1 ASCO

Commit message: bugfix
Parts:
- removed the U2 at (138.2, 81.5)
Routing:
- net +5V: track 70.5 -> 78.0 mm
- net Net-(U1-VBUS): track 2.50 -> 4.76 mm
